File: PCB_files_kicad/project/blupill.sch (KiCad schematic (older format))
At the start: 1 part, among them U4 BluePill_Connector

Commit message: PCB - Placing components
Parts:
- U4: footprint (none) -> mylib:bluepill
Changed lines of the file:
@@
 F 0 "U4" H 4575 4415 50  0000 C CNN
 F 1 "BluePill_Connector" H 4575 4324 50  0000 C CNN
-F 2 "" H 4550 4250 50  0001 C CNN
+F 2 "mylib:bluepill" H 4550 4250 50  0001 C CNN
 F 3 "" H 4550 4250 50  0001 C CNN
 	1    4550 2750

Commit message: Sche rev 1.4 - PCB rev 1.2
Connections:
- net L3_GPIO: now also U4.19 (PA5); no longer U4.21 (PA6)
- net L4_GPIO: now also U4.21 (PA6); no longer U4.19 (PA5)
Changed lines of the file:
@@
 Sheet 3 3
 Title "Sistema de Alarma"
-Date "2021-09-15"
-Rev "v1.2"
+Date "2021-09-23"
+Rev "v1.4"
 Comp "Proyecto Técnicas Digitales II - Grupo N°4"
 Comment1 "Liaño, Lucas"
@@
 Wire Wire Line
 	4050 2750 3550 2750
-Text HLabel 3550 2900 0    59   Output ~ 0
-L3_GPIO
 Text HLabel 3550 2750 0    59   Output ~ 0
+L3_GPIO
+Text HLabel 3550 2900 0    59   Output ~ 0
 L4_GPIO
 Wire Wire Line

Commit message: Schematic v1.7 - PCB v1.4
Parts:
- renumbered U4 to U5
Changed lines of the file:
@@
 Sheet 3 3
 Title "Sistema de Alarma"
-Date "2021-09-27"
-Rev "v1.6"
+Date "2021-09-29"
+Rev "v1.7"
 Comp "Proyecto Técnicas Digitales II - Grupo N°4"
 Comment1 "Liaño, Lucas"
@@
 P 4550 2750
 AR Path="/60FADDA4" Ref="U?"  Part="1"
-AR Path="/60FAC4BE/60FADDA4" Ref="U4"  Part="1"
-F 0 "U4" H 4575 4415 50  0000 C CNN
+AR Path="/60FAC4BE/60FADDA4" Ref="U5"  Part="1"
+F 0 "U5" H 4575 4415 50  0000 C CNN
 F 1 "BluePill_Connector" H 4575 4324 50  0000 C CNN
 F 2 "mylib:bluepill" H 4550 4250 50  0001 C CNN
@@
 	3700 4250 3700 4550
 $Comp
-L power:GND #PWR0117
+L power:GND #PWR044
 U 1 1 612C500D
 P 3700 4550
-F 0 "#PWR0117" H 3700 4300 50  0001 C CNN
+F 0 "#PWR044" H 3700 4300 50  0001 C CNN
 F 1 "GND" H 3705 4377 50  0000 C CNN
 F 2 "" H 3700 4550 50  0001 C CNN
@@
 	6300 1550 6300 1650
 $Comp
-L power:GND #PWR0118
+L power:GND #PWR045
 U 1 1 612C5FE6
 P 6300 1650
-F 0 "#PWR0118" H 6300 1400 50  0001 C CNN
+F 0 "#PWR045" H 6300 1400 50  0001 C CNN
 F 1 "GND" H 6305 1477 50  0000 C CNN
 F 2 "" H 6300 1650 50  0001 C CNN

Commit message: Minor changes
Connections:
- net OUTPUT_3V3: no longer U5.2 (+3.3V), U5.35 (+3.3V)
- no-connect marks 10 -> 12
Changed lines of the file:
@@
 EndData
 $EndBitmap
-NoConn ~ 4050 3800
 $Comp
 L myLib:BluePill_Connector U?
@@
 Wire Wire Line
 	5400 1700 5100 1700
-Wire Wire Line
-	4050 3950 3700 3950
 Text Label 5400 1700 0    50   ~ 0
 5V
-Text Label 5400 1400 0    50   ~ 0
-3V3
-Text Label 3700 3950 2    50   ~ 0
-3V3
 Wire Wire Line
 	4050 4100 3700 4100
@@
 	3700 4250 3700 4550
 $Comp
-L power:GND #PWR044
+L power:GND #PWR045
 U 1 1 612C500D
 P 3700 4550
-F 0 "#PWR044" H 3700 4300 50  0001 C CNN
+F 0 "#PWR045" H 3700 4300 50  0001 C CNN
 F 1 "GND" H 3705 4377 50  0000 C CNN
 F 2 "" H 3700 4550 50  0001 C CNN
@@
 	6300 1550 6300 1650
 $Comp
-L power:GND #PWR045
+L power:GND #PWR046
 U 1 1 612C5FE6
 P 6300 1650
-F 0 "#PWR045" H 6300 1400 50  0001 C CNN
+F 0 "#PWR046" H 6300 1400 50  0001 C CNN
 F 1 "GND" H 6305 1477 50  0000 C CNN
 F 2 "" H 6300 1650 50  0001 C CNN
@@
 Power
 Wire Wire Line
-	5100 1400 5400 1400
-Wire Wire Line
 	4050 3500 3550 3500
 Text HLabel 3550 3350 0    59   Output ~ 0
@@
 Text Label 3700 1400 2    50   ~ 0
 3V3
+NoConn ~ 4050 3950
+NoConn ~ 5100 1400
+NoConn ~ 4050 3800
 $EndSCHEMATC
