File: PCB_files_kicad/project/power.sch (KiCad schematic (older format))
At the start: 27 parts, among them J7 Barrel_Jack, J8 USB_B_Micro, Q1 IRF9Z20, U2 TP4056, U3 LM1117-3.3, U4 MT3608

Commit message: Minor changes
Parts:
- added C2: 10uF, Capacitor_SMD:C_0805_2012Metric_Pad1.18x1.45mm_HandSolder, symbol Device:C
- renumbered C2 to C3, C3 to C4, C4 to C5, C5 to C6
Connections:
- net Earth: now also C2.2
- net OUTPUT_5V: now also C2.1
Changed lines of the file:
@@
 P 4150 4400
 AR Path="/60FAC4BE/6100EABA" Ref="#PWR?"  Part="1"
-AR Path="/60FFCFF1/6100EABA" Ref="#PWR034"  Part="1"
-F 0 "#PWR034" H 4150 4150 50  0001 C CNN
+AR Path="/60FFCFF1/6100EABA" Ref="#PWR035"  Part="1"
+F 0 "#PWR035" H 4150 4150 50  0001 C CNN
 F 1 "Earth" H 4150 4250 50  0001 C CNN
 F 2 "" H 4150 4400 50  0001 C CNN
@@
 P 4850 2900
 AR Path="/60FAC4BE/61029C39" Ref="#PWR?"  Part="1"
-AR Path="/60FFCFF1/61029C39" Ref="#PWR037"  Part="1"
-F 0 "#PWR037" H 4850 2650 50  0001 C CNN
+AR Path="/60FFCFF1/61029C39" Ref="#PWR038"  Part="1"
+F 0 "#PWR038" H 4850 2650 50  0001 C CNN
 F 1 "Earth" H 4850 2750 50  0001 C CNN
 F 2 "" H 4850 2900 50  0001 C CNN
@@
 P 8450 3800
 AR Path="/60FAC4BE/6102A554" Ref="C?"  Part="1"
-AR Path="/60FFCFF1/6102A554" Ref="C5"  Part="1"
-F 0 "C5" H 8500 3900 50  0000 L CNN
+AR Path="/60FFCFF1/6102A554" Ref="C6"  Part="1"
+F 0 "C6" H 8500 3900 50  0000 L CNN
 F 1 "22uF" H 8500 3700 50  0000 L CNN
 F 2 "Capacitor_THT:CP_Radial_D5.0mm_P2.50mm" H 8488 3650 50  0001 C CNN
@@
 P 6050 3900
 AR Path="/60FAC4BE/61045CAF" Ref="C?"  Part="1"
-AR Path="/60FFCFF1/61045CAF" Ref="C4"  Part="1"
-F 0 "C4" H 6100 4000 50  0000 L CNN
+AR Path="/60FFCFF1/61045CAF" Ref="C5"  Part="1"
+F 0 "C5" H 6100 4000 50  0000 L CNN
 F 1 "22uF" H 6100 3800 50  0000 L CNN
 F 2 "Capacitor_THT:CP_Radial_D5.0mm_P2.50mm" H 6088 3750 50  0001 C CNN
@@
 P 6050 4650
 AR Path="/60FAC4BE/6104C10B" Ref="#PWR?"  Part="1"
-AR Path="/60FFCFF1/6104C10B" Ref="#PWR039"  Part="1"
-F 0 "#PWR039" H 6050 4400 50  0001 C CNN
+AR Path="/60FFCFF1/6104C10B" Ref="#PWR040"  Part="1"
+F 0 "#PWR040" H 6050 4400 50  0001 C CNN
 F 1 "Earth" H 6050 4500 50  0001 C CNN
 F 2 "" H 6050 4650 50  0001 C CNN
@@
 P 7050 4650
 AR Path="/60FAC4BE/6104C90C" Ref="#PWR?"  Part="1"
-AR Path="/60FFCFF1/6104C90C" Ref="#PWR040"  Part="1"
-F 0 "#PWR040" H 7050 4400 50  0001 C CNN
+AR Path="/60FFCFF1/6104C90C" Ref="#PWR041"  Part="1"
+F 0 "#PWR041" H 7050 4400 50  0001 C CNN
 F 1 "Earth" H 7050 4500 50  0001 C CNN
 F 2 "" H 7050 4650 50  0001 C CNN
@@
 P 8450 4650
 AR Path="/60FAC4BE/6104D029" Ref="#PWR?"  Part="1"
-AR Path="/60FFCFF1/6104D029" Ref="#PWR042"  Part="1"
-F 0 "#PWR042" H 8450 4400 50  0001 C CNN
+AR Path="/60FFCFF1/6104D029" Ref="#PWR043"  Part="1"
+F 0 "#PWR043" H 8450 4400 50  0001 C CNN
 F 1 "Earth" H 8450 4500 50  0001 C CNN
 F 2 "" H 8450 4650 50  0001 C CNN
@@
 P 9400 4650
 AR Path="/60FAC4BE/6126B40D" Ref="#PWR?"  Part="1"
-AR Path="/60FFCFF1/6126B40D" Ref="#PWR043"  Part="1"
-F 0 "#PWR043" H 9400 4400 50  0001 C CNN
+AR Path="/60FFCFF1/6126B40D" Ref="#PWR044"  Part="1"
+F 0 "#PWR044" H 9400 4400 50  0001 C CNN
 F 1 "Earth" H 9400 4500 50  0001 C CNN
 F 2 "" H 9400 4650 50  0001 C CNN
@@
 OUTPUT_BAT
 $Comp
-L power:PWR_FLAG #FLG04
+L power:PWR_FLAG #FLG03
 U 1 1 616505D3
 P 6550 3200
-F 0 "#FLG04" H 6550 3275 50  0001 C CNN
+F 0 "#FLG03" H 6550 3275 50  0001 C CNN
 F 1 "PWR_FLAG" H 6550 3373 50  0001 C CNN
 F 2 "" H 6550 3200 50  0001 C CNN
@@
 $EndComp
 $Comp
-L power:PWR_FLAG #FLG03
+L power:PWR_FLAG #FLG02
 U 1 1 616872FC
 P 2600 2450
-F 0 "#FLG03" H 2600 2525 50  0001 C CNN
+F 0 "#FLG02" H 2600 2525 50  0001 C CNN
 F 1 "PWR_FLAG" H 2600 2623 50  0001 C CNN
 F 2 "" H 2600 2450 50  0001 C CNN
@@
 P 5100 3600
 AR Path="/60FAC4BE/612CF008" Ref="C?"  Part="1"
-AR Path="/60FFCFF1/612CF008" Ref="C3"  Part="1"
-F 0 "C3" H 4950 3700 50  0000 L CNN
+AR Path="/60FFCFF1/612CF008" Ref="C4"  Part="1"
+F 0 "C4" H 4950 3700 50  0000 L CNN
 F 1 "10uF" H 4900 3450 50  0000 L CNN
 F 2 "Capacitor_THT:CP_Radial_D5.0mm_P2.50mm" H 5138 3450 50  0001 C CNN
@@
 P 5100 4400
 AR Path="/60FAC4BE/612CF00E" Ref="#PWR?"  Part="1"
-AR Path="/60FFCFF1/612CF00E" Ref="#PWR038"  Part="1"
-F 0 "#PWR038" H 5100 4150 50  0001 C CNN
+AR Path="/60FFCFF1/612CF00E" Ref="#PWR039"  Part="1"
+F 0 "#PWR039" H 5100 4150 50  0001 C CNN
 F 1 "Earth" H 5100 4250 50  0001 C CNN
 F 2 "" H 5100 4400 50  0001 C CNN
@@
 P 3450 4400
 AR Path="/60FAC4BE/61318E5C" Ref="#PWR?"  Part="1"
-AR Path="/60FFCFF1/61318E5C" Ref="#PWR031"  Part="1"
-F 0 "#PWR031" H 3450 4150 50  0001 C CNN
+AR Path="/60FFCFF1/61318E5C" Ref="#PWR032"  Part="1"
+F 0 "#PWR032" H 3450 4150 50  0001 C CNN
 F 1 "Earth" H 3450 4250 50  0001 C CNN
 F 2 "" H 3450 4400 50  0001 C CNN
@@
 P 4550 4400
 AR Path="/60FAC4BE/613DDC9E" Ref="#PWR?"  Part="1"
-AR Path="/60FFCFF1/613DDC9E" Ref="#PWR036"  Part="1"
-F 0 "#PWR036" H 4550 4150 50  0001 C CNN
+AR Path="/60FFCFF1/613DDC9E" Ref="#PWR037"  Part="1"
+F 0 "#PWR037" H 4550 4150 50  0001 C CNN
 F 1 "Earth" H 4550 4250 50  0001 C CNN
 F 2 "" H 4550 4400 50  0001 C CNN
@@
 P 4000 3750
 AR Path="/60FAC4BE/6142B07E" Ref="#PWR?"  Part="1"
-AR Path="/60FFCFF1/6142B07E" Ref="#PWR033"  Part="1"
-F 0 "#PWR033" H 4000 3500 50  0001 C CNN
+AR Path="/60FFCFF1/6142B07E" Ref="#PWR034"  Part="1"
+F 0 "#PWR034" H 4000 3500 50  0001 C CNN
 F 1 "Earth" H 4000 3600 50  0001 C CNN
 F 2 "" H 4000 3750 50  0001 C CNN
@@
 P 8000 4650
 AR Path="/60FAC4BE/61464B18" Ref="#PWR?"  Part="1"
-AR Path="/60FFCFF1/61464B18" Ref="#PWR041"  Part="1"
-F 0 "#PWR041" H 8000 4400 50  0001 C CNN
+AR Path="/60FFCFF1/61464B18" Ref="#PWR042"  Part="1"
+F 0 "#PWR042" H 8000 4400 50  0001 C CNN
 F 1 "Earth" H 8000 4500 50  0001 C CNN
 F 2 "" H 8000 4650 50  0001 C CNN
@@
 P 4250 5950
 AR Path="/60FAC4BE/61597DB5" Ref="C?"  Part="1"
-AR Path="/60FFCFF1/61597DB5" Ref="C2"  Part="1"
-F 0 "C2" H 4100 6050 50  0000 L CNN
+AR Path="/60FFCFF1/61597DB5" Ref="C3"  Part="1"
+F 0 "C3" H 4100 6050 50  0000 L CNN
 F 1 "10uF" H 4050 5850 50  0000 L CNN
 F 2 "Capacitor_SMD:C_0805_2012Metric_Pad1.18x1.45mm_HandSolder" H 4288 5800 50  0001 C CNN
@@
 P 3800 6450
 AR Path="/60FAC4BE/615A59FA" Ref="#PWR?"  Part="1"
-AR Path="/60FFCFF1/615A59FA" Ref="#PWR032"  Part="1"
-F 0 "#PWR032" H 3800 6200 50  0001 C CNN
+AR Path="/60FFCFF1/615A59FA" Ref="#PWR033"  Part="1"
+F 0 "#PWR033" H 3800 6200 50  0001 C CNN
 F 1 "Earth" H 3800 6300 50  0001 C CNN
 F 2 "" H 3800 6450 50  0001 C CNN
@@
 P 4250 6450
 AR Path="/60FAC4BE/615A5E03" Ref="#PWR?"  Part="1"
-AR Path="/60FFCFF1/615A5E03" Ref="#PWR035"  Part="1"
-F 0 "#PWR035" H 4250 6200 50  0001 C CNN
+AR Path="/60FFCFF1/615A5E03" Ref="#PWR036"  Part="1"
+F 0 "#PWR036" H 4250 6200 50  0001 C CNN
 F 1 "Earth" H 4250 6300 50  0001 C CNN
 F 2 "" H 4250 6450 50  0001 C CNN
@@
 Voltage Regulator 3.3V\n
 Wire Wire Line
-	3000 5450 3500 5450
+	3000 5450 3350 5450
+$Comp
+L Device:C C?
+U 1 1 61564AE1
+P 3350 5950
+AR Path="/60FAC4BE/61564AE1" Ref="C?"  Part="1"
+AR Path="/60FFCFF1/61564AE1" Ref="C2"  Part="1"
+F 0 "C2" H 3200 6050 50  0000 L CNN
+F 1 "10uF" H 3150 5850 50  0000 L CNN
+F 2 "Capacitor_SMD:C_0805_2012Metric_Pad1.18x1.45mm_HandSolder" H 3388 5800 50  0001 C CNN
+F 3 "~" H 3350 5950 50  0001 C CNN
+	1    3350 5950
+	1    0    0    -1
+$EndComp
+Wire Wire Line
+	3350 6100 3350 6450
+$Comp
+L power:Earth #PWR?
+U 1 1 61564AE9
+P 3350 6450
+AR Path="/60FAC4BE/61564AE9" Ref="#PWR?"  Part="1"
+AR Path="/60FFCFF1/61564AE9" Ref="#PWR031"  Part="1"
+F 0 "#PWR031" H 3350 6200 50  0001 C CNN
+F 1 "Earth" H 3350 6300 50  0001 C CNN
+F 2 "" H 3350 6450 50  0001 C CNN
+F 3 "~" H 3350 6450 50  0001 C CNN
+	1    3350 6450
+	1    0    0    -1
+$EndComp
+Wire Wire Line
+	3350 5800 3350 5450
+Connection ~ 3350 5450
+Wire Wire Line
+	3350 5450 3500 5450
 $EndSCHEMATC
