File: PCB_files_kicad/project/project.kicad_pcb (KiCad board)
At the start: 2 copper layers, 65 x 100 mm, 53 parts, among them J1 Conn_01x08_Female, J2 S1, J3 S2, J4 Conn_01x08_Female, J5 Display, J6 HC06, J7 Barrel_Jack, J8 USB_B_Micro, Q1 IRF9Z20, U1 M24C02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

Commit message: PCB v1.5
Other:
- board text added: "C1"
- board text added: "C2"
- board text added: "C3"
- board text added: "C4"
- board text added: "L1"
- board text added: "L2"
- board text added: "L3"
- board text added: "L4"
- board text added: "MISO"
- board text added: "MOSI"
- board text added: "NSS"
- board text added: "SCK"

Commit message: Minor changes
Parts:
- added C2: 10uF, Capacitor_SMD:C_0805_2012Metric_Pad1.18x1.45mm_HandSolder, F.Cu at (124.8, 88.0)
- moved C3 0.75 mm to (120.5, 88.0)
- renumbered C2 to C3, C3 to C4, C4 to C5, C5 to C6
Connections:
- U1 pad 8: +5V -> +3V3
- U5 pad 2: +3V3 -> Net-(U5-Pad2)
- U5 pad 35: +3V3 -> Net-(U5-Pad35)
Routing:
- net /blupill/SENSOR2_GPIO: track 47.5 -> 35.1 mm
- net +5V: track 222.6 -> 212.4 mm
- net Earth: track 27.5 -> 37.0 mm, vias 42 -> 48
- net /blupill/SENSOR1_GPIO: track 39.9 -> 31.8 mm
- net +3V3: track 224.6 -> 230.6 mm, vias 0 -> 2
- net /blupill/SPI2_SCK: track 37.1 -> 32.6 mm
- net Net-(R9-Pad2): track 42.5 -> 39.6 mm
- net /I2C1_SCL: track 98.6 -> 101.1 mm
- net /blupill/ADC12_IN1: track 60.2 -> 62.0 mm
- net /blupill/ADC12_IN0: track 53.4 -> 51.7 mm
- net Net-(R11-Pad2): track 60.2 -> 61.4 mm
