File: PCB_files_kicad/project/project.sch (KiCad schematic (older format))
At the start: 20 parts, among them J1 Conn_01x08_Female, J2 S1, J3 S2, J4 Conn_01x08_Female, J5 Display, J6 HC06, U1 24AA64FT-I/OT

Commit message: PCB - Placing components
Parts:
- BZ1: footprint (none) -> Buzzer_Beeper:Buzzer_12x9.5RM7.6
- D1: footprint (none) -> LED_THT:LED_D5.0mm; Mouser Link https://ar.mouser.com/ProductDetail/Wurth-Elektronik/150060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 -> (none); Mouser Number 710-150060VS75000 -> (none); Part Number 150060VS75000 -> (none)
- D2: footprint (none) -> LED_THT:LED_D5.0mm; Mouser Link https://ar.mouser.com/ProductDetail/Wurth-Elektronik/150060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 -> (none); Mouser Number 710-150060RS75000 -> (none); Part Number 150060RS75000 -> (none)
- H1, H2, H3, H4: footprint (none) -> MountingHole:MountingHole_3.2mm_M3_DIN965_Pad_TopBottom
- J1, J4: footprint Connector_PinHeader_2.54mm:PinHeader_1x08_P2.54mm_Horizontal -> Connector_PinHeader_2.54mm:PinHeader_1x08_P2.54mm_Vertical
- J2, J3: footprint (none) -> TerminalBlock:TerminalBlock_bornier-3_P5.08mm
- J5, J6: footprint (none) -> TerminalBlock:TerminalBlock_bornier-4_P5.08mm
- R1, R2, R5, R6, R8, R9: footprint (none) -> Resistor_THT:R_Axial_DIN0414_L11.9mm_D4.5mm_P20.32mm_Horizontal
- U1: footprint Package_TO_SOT_SMD:SOT-23-5 -> Package_TO_SOT_SMD:SOT-23-6_Handsoldering; symbol Memory_EEPROM:AT24CS01-STUM -> myLib:AT24CS01-STUM
Connections:
- no-connect marks 2 -> 3
Changed lines of the file:
@@
 F 0 "H1" H 5050 7153 50  0001 L CNN
 F 1 "MountingHole_Pad" H 5050 7108 50  0001 L CNN
-F 2 "" H 4950 7150 50  0001 C CNN
+F 2 "MountingHole:MountingHole_3.2mm_M3_DIN965_Pad_TopBottom" H 4950 7150 50  0001 C CNN
 F 3 "~" H 4950 7150 50  0001 C CNN
 	1    4950 7150
@@
 F 0 "H2" H 5300 7153 50  0001 L CNN
 F 1 "MountingHole_Pad" H 5300 7108 50  0001 L CNN
-F 2 "" H 5200 7150 50  0001 C CNN
+F 2 "MountingHole:MountingHole_3.2mm_M3_DIN965_Pad_TopBottom" H 5200 7150 50  0001 C CNN
 F 3 "~" H 5200 7150 50  0001 C CNN
 	1    5200 7150
@@
 F 0 "H3" H 5550 7153 50  0001 L CNN
 F 1 "MountingHole_Pad" H 5550 7108 50  0001 L CNN
-F 2 "" H 5450 7150 50  0001 C CNN
+F 2 "MountingHole:MountingHole_3.2mm_M3_DIN965_Pad_TopBottom" H 5450 7150 50  0001 C CNN
 F 3 "~" H 5450 7150 50  0001 C CNN
 	1    5450 7150
@@
 F 0 "H4" H 5800 7153 50  0001 L CNN
 F 1 "MountingHole_Pad" H 5800 7108 50  0001 L CNN
-F 2 "" H 5700 7150 50  0001 C CNN
+F 2 "MountingHole:MountingHole_3.2mm_M3_DIN965_Pad_TopBottom" H 5700 7150 50  0001 C CNN
 F 3 "~" H 5700 7150 50  0001 C CNN
 	1    5700 7150
@@
 F 0 "J1" H 3100 3600 50  0000 C CNN
 F 1 "Conn_01x08_Female" H 2842 3994 50  0001 C CNN
-F 2 "Connector_PinHeader_2.54mm:PinHeader_1x08_P2.54mm_Horizontal" H 2950 3600 50  0001 C CNN
+F 2 "Connector_PinHeader_2.54mm:PinHeader_1x08_P2.54mm_Vertical" H 2950 3600 50  0001 C CNN
 F 3 "~" H 2950 3600 50  0001 C CNN
 	1    2950 3600
@@
 F 0 "J2" H 3150 1950 50  0000 C CNN
 F 1 "S1" H 3150 2050 50  0000 C CNN
-F 2 "" H 3000 1950 50  0001 C CNN
+F 2 "TerminalBlock:TerminalBlock_bornier-3_P5.08mm" H 3000 1950 50  0001 C CNN
 F 3 "~" H 3000 1950 50  0001 C CNN
 	1    3000 1950
@@
 F 0 "J3" H 3150 2650 50  0000 C CNN
 F 1 "S2" H 3150 2550 50  0000 C CNN
-F 2 "" H 3000 2550 50  0001 C CNN
+F 2 "TerminalBlock:TerminalBlock_bornier-3_P5.08mm" H 3000 2550 50  0001 C CNN
 F 3 "~" H 3000 2550 50  0001 C CNN
 	1    3000 2550
@@
 F 0 "R1" V 5695 2600 50  0000 C CNN
 F 1 "100" V 5786 2600 50  0000 C CNN
-F 2 "" V 5940 2590 50  0001 C CNN
+F 2 "Resistor_THT:R_Axial_DIN0414_L11.9mm_D4.5mm_P20.32mm_Horizontal" V 5940 2590 50  0001 C CNN
 F 3 "~" H 5900 2600 50  0001 C CNN
 	1    5900 2600
@@
 F 0 "D1" H 5493 2345 50  0000 C CNN
 F 1 "LED_Green@2V" H 5493 2436 50  0000 C CNN
-F 2 "" H 5500 2600 50  0001 C CNN
-F 3 "https://ar.mouser.com/datasheet/2/445/150060VS75000-1714627.pdf" H 5500 2600 50  0001 C CNN
-F 4 "https://ar.mouser.com/ProductDetail/Wurth-Elektronik/150060VS75000?qs=LlUlMxKIyB1Q1Bi5mQ%2FKLw%3D%3D" H 5500 2600 50  0001 C CNN "Mouser Link"
-F 5 "710-150060VS75000 " H 5500 2600 50  0001 C CNN "Mouser Number"
-F 6 "150060VS75000" H 5500 2600 50  0001 C CNN "Part Number"
+F 2 "LED_THT:LED_D5.0mm" H 5500 2600 50  0001 C CNN
+F 3 "" H 5500 2600 50  0001 C CNN
+F 4 "" H 5500 2600 50  0001 C CNN "Mouser Link"
+F 5 "" H 5500 2600 50  0001 C CNN "Mouser Number"
+F 6 "" H 5500 2600 50  0001 C CNN "Part Number"
 	1    5500 2600
 	1    0    0    1
@@
 F 0 "R2" V 6395 2750 50  0000 C CNN
 F 1 "100" V 6486 2750 50  0000 C CNN
-F 2 "" V 6640 2740 50  0001 C CNN
+F 2 "Resistor_THT:R_Axial_DIN0414_L11.9mm_D4.5mm_P20.32mm_Horizontal" V 6640 2740 50  0001 C CNN
 F 3 "~" H 6600 2750 50  0001 C CNN
 	1    6600 2750
@@
 F 0 "D2" H 6350 2700 50  0000 C CNN
 F 1 "LED_Red@2V" H 6250 2850 50  0000 C CNN
-F 2 "" H 6200 2750 50  0001 C CNN
-F 3 "https://ar.mouser.com/datasheet/2/445/150060RS75000-1715052.pdf" H 6200 2750 50  0001 C CNN
-F 4 "https://ar.mouser.com/ProductDetail/Wurth-Elektronik/150060RS75000?qs=LlUlMxKIyB3QnmZ3fw%2FVCA%3D%3D" H 6200 2750 50  0001 C CNN "Mouser Link"
-F 5 " 710-150060RS75000 " H 6200 2750 50  0001 C CNN "Mouser Number"
-F 6 "150060RS75000 " H 6200 2750 50  0001 C CNN "Part Number"
+F 2 "LED_THT:LED_D5.0mm" H 6200 2750 50  0001 C CNN
+F 3 "" H 6200 2750 50  0001 C CNN
+F 4 "" H 6200 2750 50  0001 C CNN "Mouser Link"
+F 5 "" H 6200 2750 50  0001 C CNN "Mouser Number"
+F 6 "" H 6200 2750 50  0001 C CNN "Part Number"
 	1    6200 2750
 	1    0    0    1
@@
 F 0 "J5" H 7422 5124 50  0000 R CNN
 F 1 "Display" H 7422 5033 50  0000 R CNN
-F 2 "" H 7450 5150 50  0001 C CNN
+F 2 "TerminalBlock:TerminalBlock_bornier-4_P5.08mm" H 7450 5150 50  0001 C CNN
 F 3 "~" H 7450 5150 50  0001 C CNN
 	1    7450 5150
@@
 F 0 "J4" H 7250 4150 50  0000 C CNN
 F 1 "Conn_01x08_Female" H 7292 4094 50  0001 C CNN
-F 2 "Connector_PinHeader_2.54mm:PinHeader_1x08_P2.54mm_Horizontal" H 7400 3700 50  0001 C CNN
+F 2 "Connector_PinHeader_2.54mm:PinHeader_1x08_P2.54mm_Vertical" H 7400 3700 50  0001 C CNN
 F 3 "~" H 7400 3700 50  0001 C CNN
 	1    7400 3700
@@
 F 0 "BZ1" H 8952 3729 50  0000 L CNN
 F 1 "Buzzer" H 8952 3638 50  0000 L CNN
-F 2 "" V 8775 3800 50  0001 C CNN
+F 2 "Buzzer_Beeper:Buzzer_12x9.5RM7.6" V 8775 3800 50  0001 C CNN
 F 3 "~" V 8775 3800 50  0001 C CNN
 	1    8800 3700
@@
 F 0 "J6" H 9150 4950 50  0000 C CNN
 F 1 "HC06" H 9150 4850 50  0000 C CNN
-F 2 "" H 9000 4950 50  0001 C CNN
+F 2 "TerminalBlock:TerminalBlock_bornier-4_P5.08mm" H 9000 4950 50  0001 C CNN
 F 3 "~" H 9000 4950 50  0001 C CNN
 	1    9000 4950
@@
 	6800 5250 7250 5250
 $Comp
-L Memory_EEPROM:AT24CS01-STUM U1
+L myLib:AT24CS01-STUM U1
 U 1 1 615E11DA
 P 8300 2150
-F 0 "U1" H 7970 2196 50  0000 R CNN
-F 1 "24AA64FT-I/OT" H 7950 2100 50  0000 R CNN
-F 2 "Package_TO_SOT_SMD:SOT-23-5" H 8300 2150 50  0001 C CNN
+F 0 "U1" H 8100 2400 50  0000 R CNN
+F 1 "24AA64FT-I/OT" H 7950 2050 50  0000 R CNN
+F 2 "Package_TO_SOT_SMD:SOT-23-6_Handsoldering" H 8300 2150 50  0001 C CNN
 F 3 "https://ar.mouser.com/datasheet/2/268/22154B-1221207.pdf" H 8300 2150 50  0001 C CNN
 F 4 "https://ar.mouser.com/ProductDetail/Microchip-Technology/24AA64FT-I-OT?qs=WqWCsLCZBkrRsEB9Ux8Tvw%3D%3D" H 8300 2150 50  0001 C CNN "Mouser Link"
@@
 F 0 "R5" H 6418 1496 50  0000 L CNN
 F 1 "2k" H 6418 1405 50  0000 L CNN
-F 2 "" V 6390 1440 50  0001 C CNN
+F 2 "Resistor_THT:R_Axial_DIN0414_L11.9mm_D4.5mm_P20.32mm_Horizontal" V 6390 1440 50  0001 C CNN
 F 3 "~" H 6350 1450 50  0001 C CNN
 	1    6350 1450
@@
 F 0 "R6" H 6418 1896 50  0000 L CNN
 F 1 "3k" H 6418 1805 50  0000 L CNN
-F 2 "" V 6390 1840 50  0001 C CNN
+F 2 "Resistor_THT:R_Axial_DIN0414_L11.9mm_D4.5mm_P20.32mm_Horizontal" V 6390 1840 50  0001 C CNN
 F 3 "~" H 6350 1850 50  0001 C CNN
 	1    6350 1850
@@
 F 0 "R8" H 6868 1496 50  0000 L CNN
 F 1 "2k" H 6868 1405 50  0000 L CNN
-F 2 "" V 6840 1440 50  0001 C CNN
+F 2 "Resistor_THT:R_Axial_DIN0414_L11.9mm_D4.5mm_P20.32mm_Horizontal" V 6840 1440 50  0001 C CNN
 F 3 "~" H 6800 1450 50  0001 C CNN
 	1    6800 1450
@@
 F 0 "R9" H 6868 1896 50  0000 L CNN
 F 1 "3k" H 6868 1805 50  0000 L CNN
-F 2 "" V 6840 1840 50  0001 C CNN
+F 2 "Resistor_THT:R_Axial_DIN0414_L11.9mm_D4.5mm_P20.32mm_Horizontal" V 6840 1840 50  0001 C CNN
 F 3 "~" H 6800 1850 50  0001 C CNN
 	1    6800 1850
@@
 	1    0    0    -1
 $EndComp
+NoConn ~ 8700 2150
 $EndSCHEMATC

Commit message: SCH version 1.3
Parts:
- added R12, R13: 2k2, Resistor_THT:R_Axial_DIN0414_L11.9mm_D4.5mm_P20.32mm_Horizontal, symbol Device:R_US
Connections:
- net +5V: now also R12.1, R13.1
- net I2C1_SCL: now also R13.2
- net I2C1_SDA: now also R12.2
Changed lines of the file:
@@
 Sheet 1 3
 Title "Sistema de Alarma"
-Date "2021-07-23"
+Date "2021-09-15"
 Rev "v1.2"
 Comp "Proyecto Técnicas Digitales II - Grupo N°4"
@@
 Text Notes 7250 6050 0    50   ~ 0
 Nota: Estan al reves TX y RX, porque en el HC06 la indicación es que el\nRX es el de entrada, es decir que se conecta con nuestro TX.
-Wire Wire Line
-	5250 4800 5650 4800
 Text Label 5650 4800 2    50   ~ 0
 I2C1_SCL
@@
 Wire Wire Line
 	6800 5350 7250 5350
-Wire Wire Line
-	5250 4650 5650 4650
 Text Label 5650 4650 2    50   ~ 0
 I2C1_SDA
@@
 $EndComp
 NoConn ~ 8700 2150
+$Comp
+L Device:R_US R12
+U 1 1 613E9F6B
+P 6050 4450
+F 0 "R12" H 6118 4496 50  0000 L CNN
+F 1 "2k2" H 6118 4405 50  0000 L CNN
+F 2 "Resistor_THT:R_Axial_DIN0414_L11.9mm_D4.5mm_P20.32mm_Horizontal" V 6090 4440 50  0001 C CNN
+F 3 "~" H 6050 4450 50  0001 C CNN
+	1    6050 4450
+	1    0    0    -1
+$EndComp
+$Comp
+L Device:R_US R13
+U 1 1 613EBFB6
+P 6350 4450
+F 0 "R13" H 6418 4496 50  0000 L CNN
+F 1 "2k2" H 6418 4405 50  0000 L CNN
+F 2 "Resistor_THT:R_Axial_DIN0414_L11.9mm_D4.5mm_P20.32mm_Horizontal" V 6390 4440 50  0001 C CNN
+F 3 "~" H 6350 4450 50  0001 C CNN
+	1    6350 4450
+	1    0    0    -1
+$EndComp
+Wire Wire Line
+	6050 4650 6050 4600
+Wire Wire Line
+	5250 4650 6050 4650
+Wire Wire Line
+	6350 4800 6350 4600
+Wire Wire Line
+	5250 4800 6350 4800
+Wire Wire Line
+	6050 4300 6050 4200
+Wire Wire Line
+	6350 4300 6350 4200
+$Comp
+L power:+5V #PWR0141
+U 1 1 61405059
+P 6050 4200
+F 0 "#PWR0141" H 6050 4050 50  0001 C CNN
+F 1 "+5V" H 6065 4373 50  0000 C CNN
+F 2 "" H 6050 4200 50  0001 C CNN
+F 3 "" H 6050 4200 50  0001 C CNN
+	1    6050 4200
+	1    0    0    -1
+$EndComp
+$Comp
+L power:+5V #PWR0142
+U 1 1 61406B09
+P 6350 4200
+F 0 "#PWR0142" H 6350 4050 50  0001 C CNN
+F 1 "+5V" H 6365 4373 50  0000 C CNN
+F 2 "" H 6350 4200 50  0001 C CNN
+F 3 "" H 6350 4200 50  0001 C CNN
+	1    6350 4200
+	1    0    0    -1
+$EndComp
 $EndSCHEMATC

Commit message: Lot of changes.. BOM was added and UTN logo too
Parts:
- J2, J3: footprint TerminalBlock:TerminalBlock_bornier-3_P5.08mm -> Connector_PinHeader_2.54mm:PinHeader_1x03_P2.54mm_Vertical
- J5, J6: footprint TerminalBlock:TerminalBlock_bornier-4_P5.08mm -> Connector_PinHeader_2.54mm:PinHeader_1x04_P2.54mm_Vertical
- R1, R2: value 100 -> 150
Changed lines of the file:
@@
 F 0 "J2" H 3150 1950 50  0000 C CNN
 F 1 "S1" H 3150 2050 50  0000 C CNN
-F 2 "TerminalBlock:TerminalBlock_bornier-3_P5.08mm" H 3000 1950 50  0001 C CNN
+F 2 "Connector_PinHeader_2.54mm:PinHeader_1x03_P2.54mm_Vertical" H 3000 1950 50  0001 C CNN
 F 3 "~" H 3000 1950 50  0001 C CNN
 	1    3000 1950
@@
 F 0 "J3" H 3150 2650 50  0000 C CNN
 F 1 "S2" H 3150 2550 50  0000 C CNN
-F 2 "TerminalBlock:TerminalBlock_bornier-3_P5.08mm" H 3000 2550 50  0001 C CNN
+F 2 "Connector_PinHeader_2.54mm:PinHeader_1x03_P2.54mm_Vertical" H 3000 2550 50  0001 C CNN
 F 3 "~" H 3000 2550 50  0001 C CNN
 	1    3000 2550
@@
 P 5900 2600
 F 0 "R1" V 5695 2600 50  0000 C CNN
-F 1 "100" V 5786 2600 50  0000 C CNN
+F 1 "150" V 5786 2600 50  0000 C CNN
 F 2 "Resistor_THT:R_Axial_DIN0414_L11.9mm_D4.5mm_P20.32mm_Horizontal" V 5940 2590 50  0001 C CNN
 F 3 "~" H 5900 2600 50  0001 C CNN
@@
 P 6600 2750
 F 0 "R2" V 6395 2750 50  0000 C CNN
-F 1 "100" V 6486 2750 50  0000 C CNN
+F 1 "150" V 6486 2750 50  0000 C CNN
 F 2 "Resistor_THT:R_Axial_DIN0414_L11.9mm_D4.5mm_P20.32mm_Horizontal" V 6640 2740 50  0001 C CNN
 F 3 "~" H 6600 2750 50  0001 C CNN
@@
 F 0 "J5" H 7422 5124 50  0000 R CNN
 F 1 "Display" H 7422 5033 50  0000 R CNN
-F 2 "TerminalBlock:TerminalBlock_bornier-4_P5.08mm" H 7450 5150 50  0001 C CNN
+F 2 "Connector_PinHeader_2.54mm:PinHeader_1x04_P2.54mm_Vertical" H 7450 5150 50  0001 C CNN
 F 3 "~" H 7450 5150 50  0001 C CNN
 	1    7450 5150
@@
 F 0 "J6" H 9150 4950 50  0000 C CNN
 F 1 "HC06" H 9150 4850 50  0000 C CNN
-F 2 "TerminalBlock:TerminalBlock_bornier-4_P5.08mm" H 9000 4950 50  0001 C CNN
+F 2 "Connector_PinHeader_2.54mm:PinHeader_1x04_P2.54mm_Vertical" H 9000 4950 50  0001 C CNN
 F 3 "~" H 9000 4950 50  0001 C CNN
 	1    9000 4950

Commit message: Sche rev 1.4 - PCB rev 1.2
Parts:
- R1, R12, R13, R2, R5, R6, R8, R9: footprint Resistor_THT:R_Axial_DIN0414_L11.9mm_D4.5mm_P20.32mm_Horizontal -> Resistor_THT:R_Axial_DIN0309_L9.0mm_D3.2mm_P12.70mm_Horizontal
Changed lines of the file:
@@
 Sheet 1 3
 Title "Sistema de Alarma"
-Date "2021-09-15"
-Rev "v1.2"
+Date "2021-09-23"
+Rev "v1.4"
 Comp "Proyecto Técnicas Digitales II - Grupo N°4"
 Comment1 "Liaño, Lucas"
@@
 F 0 "R1" V 5695 2600 50  0000 C CNN
 F 1 "150" V 5786 2600 50  0000 C CNN
-F 2 "Resistor_THT:R_Axial_DIN0414_L11.9mm_D4.5mm_P20.32mm_Horizontal" V 5940 2590 50  0001 C CNN
+F 2 "Resistor_THT:R_Axial_DIN0309_L9.0mm_D3.2mm_P12.70mm_Horizontal" V 5940 2590 50  0001 C CNN
 F 3 "~" H 5900 2600 50  0001 C CNN
 	1    5900 2600
@@
 F 0 "R2" V 6395 2750 50  0000 C CNN
 F 1 "150" V 6486 2750 50  0000 C CNN
-F 2 "Resistor_THT:R_Axial_DIN0414_L11.9mm_D4.5mm_P20.32mm_Horizontal" V 6640 2740 50  0001 C CNN
+F 2 "Resistor_THT:R_Axial_DIN0309_L9.0mm_D3.2mm_P12.70mm_Horizontal" V 6640 2740 50  0001 C CNN
 F 3 "~" H 6600 2750 50  0001 C CNN
 	1    6600 2750
@@
 F 0 "R5" H 6418 1496 50  0000 L CNN
 F 1 "2k" H 6418 1405 50  0000 L CNN
-F 2 "Resistor_THT:R_Axial_DIN0414_L11.9mm_D4.5mm_P20.32mm_Horizontal" V 6390 1440 50  0001 C CNN
+F 2 "Resistor_THT:R_Axial_DIN0309_L9.0mm_D3.2mm_P12.70mm_Horizontal" V 6390 1440 50  0001 C CNN
 F 3 "~" H 6350 1450 50  0001 C CNN
 	1    6350 1450
@@
 F 0 "R6" H 6418 1896 50  0000 L CNN
 F 1 "3k" H 6418 1805 50  0000 L CNN
-F 2 "Resistor_THT:R_Axial_DIN0414_L11.9mm_D4.5mm_P20.32mm_Horizontal" V 6390 1840 50  0001 C CNN
+F 2 "Resistor_THT:R_Axial_DIN0309_L9.0mm_D3.2mm_P12.70mm_Horizontal" V 6390 1840 50  0001 C CNN
 F 3 "~" H 6350 1850 50  0001 C CNN
 	1    6350 1850
@@
 F 0 "R8" H 6868 1496 50  0000 L CNN
 F 1 "2k" H 6868 1405 50  0000 L CNN
-F 2 "Resistor_THT:R_Axial_DIN0414_L11.9mm_D4.5mm_P20.32mm_Horizontal" V 6840 1440 50  0001 C CNN
+F 2 "Resistor_THT:R_Axial_DIN0309_L9.0mm_D3.2mm_P12.70mm_Horizontal" V 6840 1440 50  0001 C CNN
 F 3 "~" H 6800 1450 50  0001 C CNN
 	1    6800 1450
@@
 F 0 "R9" H 6868 1896 50  0000 L CNN
 F 1 "3k" H 6868 1805 50  0000 L CNN
-F 2 "Resistor_THT:R_Axial_DIN0414_L11.9mm_D4.5mm_P20.32mm_Horizontal" V 6840 1840 50  0001 C CNN
+F 2 "Resistor_THT:R_Axial_DIN0309_L9.0mm_D3.2mm_P12.70mm_Horizontal" V 6840 1840 50  0001 C CNN
 F 3 "~" H 6800 1850 50  0001 C CNN
 	1    6800 1850
@@
 F 0 "R12" H 6118 4496 50  0000 L CNN
 F 1 "2k2" H 6118 4405 50  0000 L CNN
-F 2 "Resistor_THT:R_Axial_DIN0414_L11.9mm_D4.5mm_P20.32mm_Horizontal" V 6090 4440 50  0001 C CNN
+F 2 "Resistor_THT:R_Axial_DIN0309_L9.0mm_D3.2mm_P12.70mm_Horizontal" V 6090 4440 50  0001 C CNN
 F 3 "~" H 6050 4450 50  0001 C CNN
 	1    6050 4450
@@
 F 0 "R13" H 6418 4496 50  0000 L CNN
 F 1 "2k2" H 6418 4405 50  0000 L CNN
-F 2 "Resistor_THT:R_Axial_DIN0414_L11.9mm_D4.5mm_P20.32mm_Horizontal" V 6390 4440 50  0001 C CNN
+F 2 "Resistor_THT:R_Axial_DIN0309_L9.0mm_D3.2mm_P12.70mm_Horizontal" V 6390 4440 50  0001 C CNN
 F 3 "~" H 6350 4450 50  0001 C CNN
 	1    6350 4450

Commit message: Schematic v1.5 - PCB v1.3
Parts:
- removed U1: 24AA64FT-I/OT, Package_TO_SOT_SMD:SOT-23-6_Handsoldering, symbol myLib:AT24CS01-STUM
- added TP5: TestPoint, TestPoint:TestPoint_THTPad_D2.0mm_Drill1.0mm, symbol Connector:TestPoint
- added U1: M24C02, Package_DIP:DIP-8_W7.62mm, symbol myLib:M24C02
- BZ1: footprint Buzzer_Beeper:Buzzer_12x9.5RM7.6 -> mylib:Batt
- R5, R8: value 2k -> 2k2
- R6, R9: value 3k -> 3k3
Connections:
- net +3V3: now also TP5.1
- net +5V: now also U1.8 (VCC)
- net Earth: now also U1.1 (E0), U1.2 (E1), U1.3 (E2), U1.4 (VSS), U1.7 (~WC)
- net I2C1_SCL: now also U1.6 (SCL)
- net I2C1_SDA: now also U1.5 (SDA)
- no-connect marks 3 -> 2
Other:
- note added: "Nota: WC -> GND = Write Enable"
- note removed: "Nota: WP -> GND = Write Enable"
Changed lines of the file:
@@
 Sheet 1 3
 Title "Sistema de Alarma"
-Date "2021-09-23"
-Rev "v1.4"
+Date "2021-09-26"
+Rev "v1.5"
 Comp "Proyecto Técnicas Digitales II - Grupo N°4"
 Comment1 "Liaño, Lucas"
@@
 F 0 "BZ1" H 8952 3729 50  0000 L CNN
 F 1 "Buzzer" H 8952 3638 50  0000 L CNN
-F 2 "Buzzer_Beeper:Buzzer_12x9.5RM7.6" V 8775 3800 50  0001 C CNN
+F 2 "mylib:Batt" V 8775 3800 50  0001 C CNN
 F 3 "~" V 8775 3800 50  0001 C CNN
 	1    8800 3700
@@
 Wire Wire Line
 	6800 5250 7250 5250
-$Comp
-L myLib:AT24CS01-STUM U1
-U 1 1 615E11DA
-P 8300 2150
-F 0 "U1" H 8100 2400 50  0000 R CNN
-F 1 "24AA64FT-I/OT" H 7950 2050 50  0000 R CNN
-F 2 "Package_TO_SOT_SMD:SOT-23-6_Handsoldering" H 8300 2150 50  0001 C CNN
-F 3 "https://ar.mouser.com/datasheet/2/268/22154B-1221207.pdf" H 8300 2150 50  0001 C CNN
-F 4 "https://ar.mouser.com/ProductDetail/Microchip-Technology/24AA64FT-I-OT?qs=WqWCsLCZBkrRsEB9Ux8Tvw%3D%3D" H 8300 2150 50  0001 C CNN "Mouser Link"
-F 5 "579-24AA64FT-I/OT " H 8300 2150 50  0001 C CNN "Mouser Number"
-F 6 "24AA64FT-I/OT " H 8300 2150 50  0001 C CNN "Part Number"
-	1    8300 2150
-	-1   0    0    -1
-$EndComp
 Wire Notes Line
 	9300 2900 7150 2900
@@
 EEPROM
 Text Notes 7200 2850 0    47   Italic 0
-Nota: WP -> GND = Write Enable
+Nota: WC -> GND = Write Enable
 Text Label 7450 2150 0    50   ~ 0
 I2C1_SCL
@@
 P 6350 1450
 F 0 "R5" H 6418 1496 50  0000 L CNN
-F 1 "2k" H 6418 1405 50  0000 L CNN
+F 1 "2k2" H 6418 1405 50  0000 L CNN
 F 2 "Resistor_THT:R_Axial_DIN0309_L9.0mm_D3.2mm_P12.70mm_Horizontal" V 6390 1440 50  0001 C CNN
 F 3 "~" H 6350 1450 50  0001 C CNN
@@
 P 6350 1850
 F 0 "R6" H 6418 1896 50  0000 L CNN
-F 1 "3k" H 6418 1805 50  0000 L CNN
+F 1 "3k3" H 6418 1805 50  0000 L CNN
 F 2 "Resistor_THT:R_Axial_DIN0309_L9.0mm_D3.2mm_P12.70mm_Horizontal" V 6390 1840 50  0001 C CNN
 F 3 "~" H 6350 1850 50  0001 C CNN
@@
 P 6800 1450
 F 0 "R8" H 6868 1496 50  0000 L CNN
-F 1 "2k" H 6868 1405 50  0000 L CNN
+F 1 "2k2" H 6868 1405 50  0000 L CNN
 F 2 "Resistor_THT:R_Axial_DIN0309_L9.0mm_D3.2mm_P12.70mm_Horizontal" V 6840 1440 50  0001 C CNN
 F 3 "~" H 6800 1450 50  0001 C CNN
@@
 P 6800 1850
 F 0 "R9" H 6868 1896 50  0000 L CNN
-F 1 "3k" H 6868 1805 50  0000 L CNN
+F 1 "3k3" H 6868 1805 50  0000 L CNN
 F 2 "Resistor_THT:R_Axial_DIN0309_L9.0mm_D3.2mm_P12.70mm_Horizontal" V 6840 1840 50  0001 C CNN
 F 3 "~" H 6800 1850 50  0001 C CNN
@@
 	1    0    0    -1
 $EndComp
-NoConn ~ 8700 2150
 $Comp
 L Device:R_US R12
@@
 	1    0    0    -1
 $EndComp
+$Comp
+L myLib:M24C02 U1
+U 1 1 6151E4DA
+P 8300 2150
+F 0 "U1" H 8050 1900 50  0000 C CNN
+F 1 "M24C02" H 8100 2400 50  0000 C CNN
+F 2 "Package_DIP:DIP-8_W7.62mm" H 8300 2500 50  0001 C CNN
+F 3 "http://www.st.com/content/ccc/resource/technical/document/datasheet/b0/d8/50/40/5a/85/49/6f/DM00071904.pdf/files/DM00071904.pdf/jcr:content/translations/en.DM00071904.pdf" H 8350 1650 50  0001 C CNN
+	1    8300 2150
+	-1   0    0    -1
+$EndComp
+Wire Wire Line
+	8700 2050 8850 2050
+Wire Wire Line
+	8850 2050 8850 2150
+Wire Wire Line
+	8850 2250 8700 2250
+Wire Wire Line
+	8700 2150 8850 2150
+Connection ~ 8850 2150
+Wire Wire Line
+	8850 2150 8850 2250
+Wire Wire Line
+	9000 2150 9000 2400
+Wire Wire Line
+	8850 2150 9000 2150
+$Comp
+L power:GND #PWR0143
+U 1 1 6152DE2B
+P 9000 2400
+F 0 "#PWR0143" H 9000 2150 50  0001 C CNN
+F 1 "GND" H 9005 2227 50  0001 C CNN
+F 2 "" H 9000 2400 50  0001 C CNN
+F 3 "" H 9000 2400 50  0001 C CNN
+	1    9000 2400
+	1    0    0    -1
+$EndComp
+$Comp
+L Connector:TestPoint TP5
+U 1 1 615EDBC5
+P 5900 1800
+F 0 "TP5" H 5850 2000 50  0000 L CNN
+F 1 "TestPoint" H 5958 1827 50  0001 L CNN
+F 2 "TestPoint:TestPoint_THTPad_D2.0mm_Drill1.0mm" H 6100 1800 50  0001 C CNN
+F 3 "~" H 6100 1800 50  0001 C CNN
+	1    5900 1800
+	1    0    0    -1
+$EndComp
+Wire Wire Line
+	5750 1900 5900 1900
+Wire Wire Line
+	5900 1900 5900 1800
+Connection ~ 5750 1900
 $EndSCHEMATC

Commit message: Schematic v1.7 - PCB v1.4
Parts:
- TP1: renamed from TP5; value TestPoint -> +3.3V
- renumbered R12 to R2, R5 to R3, R6 to R4, R13 to R5, R2 to R6, R8 to R7, R9 to R8

Commit message: Minor changes
Connections:
- net +3V3: now also U1.8 (VCC)
- net +5V: no longer U1.8 (VCC)
Changed lines of the file:
@@
 	3200 1950 4000 1950
 $Comp
-L power:+5V #PWR02
+L power:+5V #PWR03
 U 1 1 613FF598
 P 3300 1750
-F 0 "#PWR02" H 3300 1600 50  0001 C CNN
+F 0 "#PWR03" H 3300 1600 50  0001 C CNN
 F 1 "+5V" H 3200 1850 50  0000 C CNN
 F 2 "" H 3300 1750 50  0001 C CNN
@@
 $EndComp
 $Comp
-L power:+5V #PWR03
+L power:+5V #PWR04
 U 1 1 613FFC5D
 P 3300 2350
-F 0 "#PWR03" H 3300 2200 50  0001 C CNN
+F 0 "#PWR04" H 3300 2200 50  0001 C CNN
 F 1 "+5V" H 3200 2450 50  0000 C CNN
 F 2 "" H 3300 2350 50  0001 C CNN
@@
 $EndComp
 $Comp
-L power:GND #PWR04
+L power:GND #PWR05
 U 1 1 6140B0AA
 P 3500 2150
-F 0 "#PWR04" H 3500 1900 50  0001 C CNN
+F 0 "#PWR05" H 3500 1900 50  0001 C CNN
 F 1 "GND" H 3505 1977 50  0001 C CNN
 F 2 "" H 3500 2150 50  0001 C CNN
@@
 	4000 1950 4000 2350
 $Comp
-L power:GND #PWR05
+L power:GND #PWR06
 U 1 1 61409F32
 P 3500 2750
-F 0 "#PWR05" H 3500 2500 50  0001 C CNN
+F 0 "#PWR06" H 3500 2500 50  0001 C CNN
 F 1 "GND" H 3505 2577 50  0001 C CNN
 F 2 "" H 3500 2750 50  0001 C CNN
@@
 Wire Notes Line
 	9300 2900 7150 2900
-Wire Notes Line
-	7150 2900 7150 1500
-Wire Notes Line
-	7150 1500 9300 1500
-Wire Notes Line
-	9300 1500 9300 2900
 Wire Wire Line
 	8300 1850 8300 1700
 Wire Wire Line
 	8300 2450 8300 2550
-$Comp
-L power:+5V #PWR023
-U 1 1 6161D033
-P 8300 1700
-F 0 "#PWR023" H 8300 1550 50  0001 C CNN
-F 1 "+5V" H 8200 1800 50  0000 C CNN
-F 2 "" H 8300 1700 50  0001 C CNN
-F 3 "" H 8300 1700 50  0001 C CNN
-	1    8300 1700
-	1    0    0    -1
-$EndComp
 $Comp
 L power:GND #PWR024
@@
 $EndComp
 $Comp
-L power:PWR_FLAG #FLG02
+L power:PWR_FLAG #FLG01
 U 1 1 61497233
 P 3950 7450
-F 0 "#FLG02" H 3950 7525 50  0001 C CNN
+F 0 "#FLG01" H 3950 7525 50  0001 C CNN
 F 1 "PWR_FLAG" H 3950 7623 50  0000 C CNN
 F 2 "" H 3950 7450 50  0001 C CNN
@@
 	3250 7500 3250 7050
 $Comp
-L power:+3V3 #PWR0101
+L power:+3V3 #PWR02
 U 1 1 61603C70
 P 3250 7050
-F 0 "#PWR0101" H 3250 6900 50  0001 C CNN
+F 0 "#PWR02" H 3250 6900 50  0001 C CNN
 F 1 "+3V3" H 3265 7223 50  0000 C CNN
 F 2 "" H 3250 7050 50  0001 C CNN
@@
 	1    0    0    -1
 $EndComp
+$Comp
+L power:+3V3 #PWR?
+U 1 1 6158619C
+P 8300 1700
+F 0 "#PWR?" H 8300 1550 50  0001 C CNN
+F 1 "+3V3" H 8315 1873 50  0000 C CNN
+F 2 "" H 8300 1700 50  0001 C CNN
+F 3 "" H 8300 1700 50  0001 C CNN
+	1    8300 1700
+	1    0    0    -1
+$EndComp
+Wire Notes Line
+	7150 1450 9300 1450
+Wire Notes Line
+	9300 1450 9300 2900
+Wire Notes Line
+	7150 1450 7150 2900
 $EndSCHEMATC
