File: PCB/project/project.kicad_pcb (KiCad board)
At the start: 2 copper layers, 65 x 100 mm, 54 parts, among them J1 Conn_01x08_Female, J2 S1, J3 S2, J4 Conn_01x08_Female, J5 Display, J6 HC06, J7 Barrel_Jack, J8 USB_B_Micro, Q1 IRF9Z20, U1 M24C02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

Commit message: PCB mini bug fix
Routing:
- net /MEASURE: track 162.9 -> 163.9 mm
